File: swarmbot.kicad_sch (KiCad schematic)
At the start: 0 parts

Commit message: added microcontroller, IR transmitter, IR receiver
Parts:
- added D1: LED, symbol Device:LED
- added R1: R_Small_US, symbol Device:R_Small_US
- added U1: ATtiny85-20P, Package_DIP:DIP-8_W7.62mm, symbol MCU_Microchip_ATtiny:ATtiny85-20P
- added U2: TSOP382xx, OptoDevice:Vishay_MINICAST-3Pin, symbol Interface_Optical:TSOP382xx
Connections:
- new net: R1.1, U1.1 (~{RESET}/PB5)
- new net: U1.3 (XTAL2/PB4), U2.1 (OUT)
- new net: D1.1 (K), U1.4 (GND), U2.2 (GND)
- new net: U1.8 (VCC), U2.3 (Vs)
- new net: D1.2 (A), R1.2
